Commit message: exported better urdf I think

File: urdf/shipbot_urdf.urdf (robot description, URDF)
Before this commit: robot shipbot_urdf, 6 links, 5 joints
Links:
- link link0: mass 0.159501817678804 -> 0.159501817678803
- link link1: mass 0.236983679127427 -> 0.236983684615599
- link link2: mass 0.266489933106212 -> 0.106988184234906
- link link3: mass 0.282526325354187 -> 0.442028154005472
- link link4: mass 0.236983679120407 -> 0.236983684646082
Joints:
- joint rotary1: axis 0 0 0 -> 0 0 1; limit lower=0 upper=0 effort=0 velocity=0 -> lower=-1.57 upper=1.57 effort=7 velocity=2; origin xyz=0 -0.01605 0 rpy=0 0 -3.1416 -> xyz=0 0 0 rpy=3.1416 1.5708 0; type fixed -> revolute
- joint rotary2: axis 0 0 0 -> 0 0 1; limit lower=0 upper=0 effort=0 velocity=0 -> lower=-1.57 upper=1.57 effort=7 velocity=2.2; origin xyz=0.0685499999999988 0.0550000000000011 0 rpy=1.5707963267949 -0.785398163397442 1.57079632679491 -> xyz=0 0 0 rpy=0 0 3.1416; type fixed -> revolute
- joint rotary3: axis 0 0 0 -> 0 0 1; limit (none) -> lower=-1.57 upper=1.57 effort=7 velocity=2.2; origin xyz=0.425 0 -0.0310500000000005 rpy=3.14159265358979 0 -2.35619449019234 -> xyz=0 0 0 rpy=3.1416 0 3.1416; type fixed -> revolute
- joint rotary4: axis 0 0 0 -> 0 0 1; limit (none) -> lower=-1.57 upper=1.57 effort=7 velocity=2.2; origin xyz=-0.427499999999995 0 -0.0860499999999999 rpy=1.5707963267949 0 1.5707963267949 -> xyz=0 0 0 rpy=1.5708 0 1.5708; type fixed -> revolute
- joint rotary5: axis 0 0 0 -> 0 0 1; limit (none) -> lower=-1.57 upper=1.57 effort=7 velocity=2.2; origin xyz=0 0 -0.01605 rpy=3.1416 0 -0.3927 -> xyz=0 0 0 rpy=3.1416 0 -0.3927; type fixed -> revolute

Commit message: added actual urdf

File: urdf/shipbot_urdf.urdf (robot description, URDF)
Before this commit: robot shipbot, 6 links, 5 joints
Links:
- link link0: mass 0.159501817678803 -> 0.1595; geometry collision mesh filename=package://shipbot_urdf/meshes/link0.STL; visual mesh filename=package://shipbot_urdf/meshes/link0.STL
- link link1: mass 0.236983684615599 -> 0.23698; geometry collision mesh filename=package://shipbot_urdf/meshes/link1.STL; visual mesh filename=package://shipbot_urdf/meshes/link1.STL
- link link2: mass 0.106988184234906 -> 0.10699; geometry collision mesh filename=package://shipbot_urdf/meshes/link2.STL; visual mesh filename=package://shipbot_urdf/meshes/link2.STL
- link link3: mass 0.442028154005472 -> 0.44203; geometry collision mesh filename=package://shipbot_urdf/meshes/link3.STL; visual mesh filename=package://shipbot_urdf/meshes/link3.STL
- link link4: mass 0.236983684646082 -> 0.23698; geometry collision mesh filename=package://shipbot_urdf/meshes/link4.STL; visual mesh filename=package://shipbot_urdf/meshes/link4.STL
- link link5: mass 0.0222650078147918 -> 0.022265; geometry collision mesh filename=package://shipbot_urdf/meshes/link5.STL; visual mesh filename=package://shipbot_urdf/meshes/link5.STL
Joints:
- joint rotary1: origin xyz=0 0 0 rpy=3.1416 1.5708 0 -> xyz=0 0 0 rpy=0 0 0; type revolute -> continuous
- joint rotary2: origin xyz=0 0 0 rpy=0 0 3.1416 -> xyz=-0.06803 -0.00048045 0.070706 rpy=-1.5708 0 1.5708; type revolute -> continuous
- joint rotary3: origin xyz=0 0 0 rpy=3.1416 0 3.1416 -> xyz=0.425 0 -0.03105 rpy=3.1416 0 3.1416; type revolute -> continuous
- joint rotary4: origin xyz=0 0 0 rpy=1.5708 0 1.5708 -> xyz=-0.375 0 -0.03 rpy=3.1416 0 3.1416; type revolute -> continuous
- joint rotary5: origin xyz=0 0 0 rpy=3.1416 0 -0.3927 -> xyz=0.06855 0 0.05605 rpy=0 1.5708 0; type revolute -> continuous
