Commit message: Renamed robot in urdf to shipbot

File: urdf/shipbot.urdf (robot description, URDF)
Before this commit: robot shipbot_urdf, 6 links, 5 joints
Links:
- link link0: geometry visual mesh filename=package://shipbot_urdf/meshes/link0.STL
- link link1: geometry visual mesh filename=package://shipbot_urdf/meshes/link1.STL
- link link2: geometry visual mesh filename=package://shipbot_urdf/meshes/link2.STL
- link link3: geometry visual mesh filename=package://shipbot_urdf/meshes/link3.STL
- link link4: geometry visual mesh filename=package://shipbot_urdf/meshes/link4.STL
- link link5: geometry visual mesh filename=package://shipbot_urdf/meshes/link5.STL

Commit message: Added world link for gazebo spawning

File: urdf/shipbot.urdf (robot description, URDF)
Before this commit: robot shipbot, 6 links, 5 joints
Links:
- added link world
Joints:
- added joint world_to_link0: type fixed, parent world, child link0, origin xyz=0 0 0.025 rpy=0 0 0

Commit message: Added end-effector frame

File: urdf/shipbot.urdf (robot description, URDF)
Before this commit: robot shipbot, 7 links, 6 joints
Links:
- added link end_effector
Joints:
- added joint link5_to_end_effector: type fixed, parent link5, child end_effector, origin xyz=0 0 0.044386 rpy=0 0 0

Commit message: Updated link lengths

File: urdf/shipbot.urdf (robot description, URDF)
Before this commit: robot shipbot, 8 links, 7 joints
Joints:
- joint rotary3: origin xyz=0.425 0 -0.03105 rpy=3.1416 0 3.1416 -> xyz=0.4064 0 -0.03105 rpy=3.1416 0 3.1416
- joint rotary4: origin xyz=-0.375 0 -0.03 rpy=3.1416 0 3.1416 -> xyz=-0.3302 0 -0.03 rpy=3.1416 0 3.1416
- joint world_to_link0: origin xyz=0 0 0.025 rpy=0 0 0 -> xyz=0 0 0.0889 rpy=0 0 0

Commit message: Updated urdf with actual robot joint names

File: urdf/shipbot.urdf (robot description, URDF)
Before this commit: robot shipbot, 8 links, 7 joints
Joints:
- removed joint rotary1
- removed joint rotary2
- removed joint rotary3
- removed joint rotary4
- removed joint rotary5
- added joint elbow: type continuous, parent link2, child link3, origin xyz=0.4064 0 -0.03105 rpy=3.1416 0 3.1416, axis 0 0 1, limit lower=-1.57 upper=1.57 effort=7 velocity=2.2
- added joint shoulder1: type continuous, parent link0, child link1, origin xyz=0 0 0 rpy=0 0 0, axis 0 0 1, limit lower=-1.57 upper=1.57 effort=7 velocity=2
- added joint shoulder2: type continuous, parent link1, child link2, origin xyz=-0.06803 -0.00048045 0.070706 rpy=-1.5708 0 1.5708, axis 0 0 1, limit lower=-1.57 upper=1.57 effort=7 velocity=2.2
- added joint wrist1: type continuous, parent link3, child link4, origin xyz=-0.3302 0 -0.03 rpy=3.1416 0 3.1416, axis 0 0 1, limit lower=-1.57 upper=1.57 effort=7 velocity=2.2
- added joint wrist2: type continuous, parent link4, child link5, origin xyz=0.06855 0 0.05605 rpy=0 1.5708 0, axis 0 0 1, limit lower=-1.57 upper=1.57 effort=7 velocity=2.2

Commit message: Fixed merge bugs

File: urdf/shipbot.urdf (robot description, URDF)
Before this commit: robot shipbot, 10 links, 10 joints
Links:
- link end_effector: mass None -> 0.0222650078147918; geometry collision mesh filename=package://shipbot_urdf/meshes/end_effector.STL; visual mesh filename=package://shipbot_urdf/meshes/end_effector.STL
Joints:
- removed joint link5_to_end_effector

Commit message: Updated meshes and added ee_tip frame

File: urdf/shipbot.urdf (robot description, URDF)
Before this commit: robot shipbot, 10 links, 9 joints
Links:
- added link ee_tip
Joints:
- added joint ee_to_tip: type fixed, parent end_effector, child ee_tip, origin xyz=4.4386e-02 0 0 rpy=0 0 0

Commit message: updated urdf with separate links for modules and brackets and tubes

File: urdf/shipbot.urdf (robot description, URDF)
Before this commit: robot shipbot, 7 links, 6 joints
Links:
- removed link link0
- removed link link1
- removed link link2
- removed link link3
- removed link link4
- removed link link5
- removed link world
- added link elbow, mass 0.15950182865601; collision mesh filename=package://shipbot_urdf/meshes/elbow.STL; visual mesh filename=package://shipbot_urdf/meshes/elbow.STL
- added link end_effector, mass 0.0222650078147918; collision mesh filename=package://shipbot_urdf/meshes/end_effector.STL; visual mesh filename=package://shipbot_urdf/meshes/end_effector.STL
- added link lower_arm, mass 0.123024502209737; collision mesh filename=package://shipbot_urdf/meshes/lower_arm.STL; visual mesh filename=package://shipbot_urdf/meshes/lower_arm.STL
- added link shoulder1, mass 0.1595; collision mesh filename=package://shipbot_urdf/meshes/shoulder1.STL; visual mesh filename=package://shipbot_urdf/meshes/shoulder1.STL
- added link shoulder2, mass 0.15950182865601; collision mesh filename=package://shipbot_urdf/meshes/shoulder2.STL; visual mesh filename=package://shipbot_urdf/meshes/shoulder2.STL
- added link shoulder_bracket, mass 0.0774818559595891; collision mesh filename=package://shipbot_urdf/meshes/shoulder_bracket.STL; visual mesh filename=package://shipbot_urdf/meshes/shoulder_bracket.STL
- added link upper_arm, mass 0.106988184234906; collision mesh filename=package://shipbot_urdf/meshes/upper_arm.STL; visual mesh filename=package://shipbot_urdf/meshes/upper_arm.STL
- added link wrist1, mass 0.159501823139725; collision mesh filename=package://shipbot_urdf/meshes/wrist1.STL; visual mesh filename=package://shipbot_urdf/meshes/wrist1.STL
- added link wrist2, mass 0.159501828686492; collision mesh filename=package://shipbot_urdf/meshes/wrist2.STL; visual mesh filename=package://shipbot_urdf/meshes/wrist2.STL
- added link wrist_bracket, mass 0.0774818559595891; collision mesh filename=package://shipbot_urdf/meshes/wrist_bracket.STL; visual mesh filename=package://shipbot_urdf/meshes/wrist_bracket.STL
Joints:
- removed joint rotary1
- removed joint rotary2
- removed joint rotary3
- removed joint rotary4
- removed joint rotary5
- removed joint world_to_link0
- added joint bracket_to_wrist2: type fixed, parent wrist_bracket, child wrist2, origin xyz=0.038 0 0.05605 rpy=0 1.5708 0, axis 0 0 0
- added joint elbow_joint: type continuous, parent upper_arm, child elbow, origin xyz=0.425 0 0 rpy=0 0 0, axis 0 0 1, limit lower=-1.57 upper=1.57 effort=7 velocity=2
- added joint elbow_to_lower_arm: type fixed, parent elbow, child lower_arm, origin xyz=0 0 -0.0295 rpy=0 0 0, axis 0 0 0
- added joint lower_arm_to_wrist1: type fixed, parent lower_arm, child wrist1, origin xyz=0.375 0 0 rpy=0 0 0, axis 0 0 0
- added joint shoulder1_joint: type continuous, parent shoulder1, child shoulder_bracket, origin xyz=0 0 0.0295 rpy=0 0 0, axis 0 0 1, limit lower=-1.57 upper=1.57 effort=7 velocity=2
- added joint shoulder2_joint: type continuous, parent shoulder2, child upper_arm, origin xyz=0 0 0.0295 rpy=0 0 0, axis 0 0 1, limit lower=-1.57 upper=1.57 effort=7 velocity=2
- added joint shoulder_bracket_to_shoulder2: type fixed, parent shoulder_bracket, child shoulder2, origin xyz=-0.038 0 0.05605 rpy=-1.5708 0 1.5708, axis 0 0 0
- added joint wrist1_joint: type continuous, parent wrist1, child wrist_bracket, origin xyz=0 0 0.0295 rpy=0 0 0, axis 0 0 1, limit lower=-1.57 upper=1.57 effort=7 velocity=2
- added joint wrist2_joint: type continuous, parent wrist2, child end_effector, origin xyz=0 0 0.03055 rpy=0 0 0, axis 0 0 1, limit lower=-1.57 upper=1.57 effort=7 velocity=2

Commit message: Updated mass values and link lengths in urdf. Still to finish up bracket measurements

File: urdf/shipbot.urdf (robot description, URDF)
Before this commit: robot shipbot, 11 links, 10 joints
Links:
- link elbow: mass 0.15950182865601 -> 0.345
- link end_effector: mass 0.0222650078147918 -> 0.154
- link lower_arm: mass 0.123024502209737 -> 0.322
- link shoulder1: mass 0.1595 -> 0.475
- link shoulder2: mass 0.15950182865601 -> 0.345
- link shoulder_bracket: mass 0.0774818559595891 -> 0.093
- link upper_arm: mass 0.106988184234906 -> 0.331
- link wrist1: mass 0.159501823139725 -> 0.345
- link wrist2: mass 0.159501828686492 -> 0.330
- link wrist_bracket: mass 0.0774818559595891 -> 0.093
Joints:
- joint bracket_to_wrist2: origin xyz=0.038 0 0.05605 rpy=0 1.5708 0 -> xyz=0.038 0 0.041275 rpy=0 1.5708 0
- joint ee_to_tip: origin xyz=4.4386e-02 0 0 rpy=0 0 0 -> xyz=0.09525 0 0 rpy=0 0 0
- joint elbow_joint: origin xyz=0.425 0 0 rpy=0 0 0 -> xyz=0.333 0 0 rpy=0 0 0
- joint lower_arm_to_wrist1: origin xyz=0.375 0 0 rpy=0 0 0 -> xyz=0.381 0 0 rpy=0 0 0
- joint shoulder_bracket_to_shoulder2: origin xyz=-0.038 0 0.05605 rpy=-1.5708 0 1.5708 -> xyz=-0.038 0 0.041275 rpy=-1.5708 0 1.5708

Commit message: Added more bracket dimensions and corrected some center of masses slightly

File: urdf/shipbot.urdf (robot description, URDF)
Before this commit: robot shipbot, 11 links, 10 joints
Joints:
- joint bracket_to_wrist2: origin xyz=0.038 0 0.041275 rpy=0 1.5708 0 -> xyz=0.0428625 0 0.041275 rpy=0 1.5708 0
- joint shoulder_bracket_to_shoulder2: origin xyz=-0.038 0 0.041275 rpy=-1.5708 0 1.5708 -> xyz=-0.0428625 0 0.041275 rpy=-1.5708 0 1.5708

Commit message: Updated measurements after switching modules around

File: urdf/shipbot.urdf (robot description, URDF)
Before this commit: robot shipbot, 11 links, 10 joints
Links:
- link shoulder1: mass 0.475 -> 0.345
- link shoulder2: mass 0.345 -> 0.475
Joints:
- joint ee_to_tip: origin xyz=0.09525 0 0 rpy=0 0 0 -> xyz=0 0 0.09525 rpy=0 0 0
- joint elbow_joint: axis 0 0 1 -> 0 0 -1; origin xyz=0.333 0 0 rpy=0 0 0 -> xyz=0.381 0 0 rpy=0 0 0
- joint elbow_to_lower_arm: origin xyz=0 0 -0.0295 rpy=0 0 0 -> xyz=0 0 -0.031 rpy=0 0 0
- joint lower_arm_to_wrist1: origin xyz=0.381 0 0 rpy=0 0 0 -> xyz=0.333 0 0 rpy=0 0 0
- joint shoulder1_joint: origin xyz=0 0 0.0295 rpy=0 0 0 -> xyz=0 0 0.031 rpy=0 0 0
- joint shoulder2_joint: origin xyz=0 0 0.0295 rpy=0 0 0 -> xyz=0 0 0.0451 rpy=0 0 0
- joint wrist1_joint: origin xyz=0 0 0.0295 rpy=0 0 0 -> xyz=0 0 0.031 rpy=0 0 0
- joint wrist2_joint: origin xyz=0 0 0.03055 rpy=0 0 0 -> xyz=0 0 0.031 rpy=0 0 0

Commit message: Updated urdf for pi offset

File: urdf/shipbot.urdf (robot description, URDF)
Before this commit: robot shipbot, 11 links, 10 joints
Joints:
- joint shoulder1_joint: origin xyz=0 0 0.031 rpy=0 0 0 -> xyz=0 0 0.031 rpy=0 0 -3.14159

Commit message: Updated urdf measurements

File: urdf/shipbot.urdf (robot description, URDF)
Before this commit: robot shipbot, 11 links, 10 joints
Joints:
- joint ee_to_tip: origin xyz=0 0 0.09525 rpy=0 0 0 -> xyz=0 0 0.085725 rpy=0 0 0
- joint shoulder_bracket_to_shoulder2: origin xyz=-0.0428625 0 0.041275 rpy=-1.5708 0 1.5708 -> xyz=-0.0428625 0 0.04 rpy=-1.5708 0 1.5708
